File: lmr16006-12v-3v3-sw-buck-conv.kicad_sch (KiCad schematic)
At the start: 0 parts

Commit message: Schematic and PCB Layout
Parts:
- added C1: 100nF, Capacitor-100nF:C0603_VJ0603Y104JXQCW1BC_C3834925, symbol Device:C
- added C2: 2.2uF, Capacitor-2.2uF:C0603_CL10A225KL8NNNC_C307463, symbol Device:C
- added C3: 22uF, Capacitor-22uF:C0603_TCC0603X5R226K100CT_C53032012, symbol Device:C
- added D1: D_Schottky, Schottky:POWERDI-123_L2_8-W1_8-LS3_7-RD-1_SS14FP_C894423, symbol Device:D_Schottky
- added J1, J2, J3, J4: Conn_01x01_Pin, Connector_PinHeader_1.00mm:PinHeader_1x01_P1.00mm_Vertical, symbol Connector:Conn_01x01_Pin
- added L1: 6.8uH, Inductor-6.8uH:IND-SMD_L4_0-W4_0_NRS4018T_NRS4018T6R8MDGJ_C222881, symbol Device:L
- added R1: 100K, Resistor_SMD:R_0603_1608Metric_Pad0.98x0.95mm_HandSolder, symbol Device:R
- added R2: 33.2K, Resistor_SMD:R_0603_1608Metric_Pad0.98x0.95mm_HandSolder, symbol Device:R
- added R3: 10K, Resistor_SMD:R_0603_1608Metric_Pad0.98x0.95mm_HandSolder, symbol Device:R
- added U1: LMR16006XDDCR, LMR16006XDDCR:SOT95P280X110-6N, symbol LMR16006XDDCR:LMR16006XDDCR
Connections:
- new net: C1.1, U1.1 (CB)
- new net: C1.2, D1.1 (K), L1.1, U1.6 (SW)
- new net: R2.2, R3.1, U1.3 (FB)
- new net: R1.2, U1.4 (SHDN)
- new net +3.3V: C3.1, J3.1 (Pin_1), L1.2, R2.1
- new net GND: C2.2, C3.2, D1.2 (A), J2.1 (Pin_1), J4.1 (Pin_1), R3.2, U1.2 (GND)
- new net VIN: C2.1, J1.1 (Pin_1), R1.1, U1.5 (VIN)
Other:
- note added: "Switching Buck Regulator"
- company: (none) -> H-Tronics
- title: (none) -> Switching Buck Converter
